File: atari_800xl/atari_chips/hardware/pokeymax4_5/fpga.kicad_sch (KiCad schematic)
At the start: 11 parts, among them J1 Conn_02x03_Odd_Even, Y1 ASE-49.152MHz

Commit message: After testing 4b first run, there are a few issues. Updated to 4b2 with: Corrected L/R output. ADC bias improvement. ADC preamp out/in- corrected. Moved silkscreen name!
git-svn-id: svn+ssh://192.168.0.3/home/svnfpga/repo/trunk@1476 d6161ac3-aae1-4d52-9b05-ea9ac36b53d3
Connections:
- net AUDL: now also U4.D9 (TB$5); no longer U4.C9 (TB$4)
- net AUDR: now also U4.C9 (TB$4); no longer U4.D9 (TB$5)
Changed lines of the file:
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@@
 		)
 	)
-	(label "AUDR"
+	(label "AUDL"
 		(at 154.94 36.83 90)
 		(effects
@@
 		)
 	)
-	(label "AUDL"
+	(label "AUDR"
 		(at 152.4 36.83 90)
 		(effects
@@
 		)
 	)
-	(hierarchical_label "AUDL"
+	(hierarchical_label "AUDR"
 		(shape input)
 		(at 152.4 19.05 90)
@@
 		)
 	)
-	(hierarchical_label "AUDR"
+	(hierarchical_label "AUDL"
 		(shape input)
 		(at 154.94 19.05 90)

Commit message: Pokeymax v4_53 as produced
git-svn-id: svn+ssh://192.168.0.3/home/svnfpga/repo/trunk@1512 d6161ac3-aae1-4d52-9b05-ea9ac36b53d3
Parts:
- added C20: 0.1uF, Capacitor_SMD:C_0402_1005Metric, symbol Device:C
- added C21: 2.2nf C0G, Capacitor_SMD:C_0402_1005Metric, symbol Device:C
- added R27: 1k, Resistor_SMD:R_0402_1005Metric, symbol Device:R
- added R30: 47, Resistor_SMD:R_0402_1005Metric, symbol Device:R
- added R31: 22, Resistor_SMD:R_0402_1005Metric, symbol Device:R
- renumbered C18 to C25, R16 to R19, R17 to R22, R18 to R23, R20 to R25, R21 to R26
Connections:
- net GND: now also C20.1
- net LIN1.A6: now also R31.1; no longer U4.A4 (T$6)
- net LIN2.A10: now also R27.1; no longer U4.M12 (B$21)
- net LIN2.A8: now also R30.2; no longer U4.L13 (BB$19)
- new net: R31.2, U4.A4 (T$6)
- new net: R30.1, U4.L13 (BB$19)
- new net ADC_IN: C21.1, R27.2, U4.M12 (B$21)
- new net AUD_VBIAS: C20.2, C21.2
Other:
- note added: "AUD_BIASED"
