File: atari_800xl/atari_chips/hardware/pokeymax4_5/fpga.kicad_sch (KiCad schematic)
At the start: 16 parts, among them J1 Conn_02x03_Odd_Even, Y1 ASE-49.152MHz

Commit message: kicad 10 upgrade
Parts:
- U4: value ~ -> (none)

Commit message: 4.55. Got AI to help me improve a few minor things. Regulator mode, extra decoupling for DAC, distances from edge, gnd/power plane switched, track spacing for a few important lines, bigger cap on 2.5v reg, shorter critical traces on 3.3v reg. Also it double checked the sallen key filter. Switched to the JLCPCB plugin for simpler part management.
Parts:
- C20: LCSC (none) -> C1525
- C21: LCSC (none) -> C2987940
- C25: LCSC (none) -> C57112
- J1: now not fitted; now left out of the parts list
- R1, R19, R2, R22: LCSC (none) -> C25804
- R23: LCSC (none) -> C21190
- R25: LCSC (none) -> C705736
- R26: LCSC (none) -> C4190
- R27: LCSC (none) -> C11702
- R30: LCSC (none) -> C137973
- R31: LCSC (none) -> C25092
- U4: LCSC (none) -> C1551099
- Y1: LCSC (none) -> C2901591
Connections:
- net unconnected-(U4-IO_UNUSED-PadE1)_1: now reaches U4.E1 (IO_UNUSED), U4.E10 (IO_UNUSED), U4.E12 (IO_UNUSED), U4.E3 (IO_UNUSED), U4.E4 (IO_UNUSED), U4.E6 (IO_UNUSED), U4.E8 (IO_UNUSED), U4.E9 (IO_UNUSED), U4.F1 (IO_UNUSED), U4.F10 (IO_UNUSED), U4.F12 (IO_UNUSED), U4.F4 (IO_UNUSED), U4.F8 (IO_UNUSED), U4.F9 (IO_UNUSED), U4.G10 (IO_UNUSED), U4.G4 (IO_UNUSED), U4.G5 (IO_UNUSED), U4.H1 (IO_UNUSED), U4.H10 (IO_UNUSED), U4.H2 (IO_UNUSED), U4.H3 (IO_UNUSED), U4.H5 (IO_UNUSED), U4.H9 (IO_UNUSED), U4.J1 (IO_UNUSED), U4.J10 (IO_UNUSED), U4.J2 (IO_UNUSED), U4.J9 (IO_UNUSED)
