File: atari_800xl/atari_chips/hardware/pokeymax4_5/pokey_pins.kicad_sch (KiCad schematic)
At the start: 4 parts, among them J2 Conn_01x14_Pin

Commit message: After testing 4b first run, there are a few issues. Updated to 4b2 with: Corrected L/R output. ADC bias improvement. ADC preamp out/in- corrected. Moved silkscreen name!
git-svn-id: svn+ssh://192.168.0.3/home/svnfpga/repo/trunk@1476 d6161ac3-aae1-4d52-9b05-ea9ac36b53d3
Parts:
- R22, R23: value 2k7 -> DNP
Changed lines of the file:
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@@
 			)
 		)
-		(property "Value" "2k7"
+		(property "Value" "DNP"
 			(at 48.26 114.2999 0)
 			(effects
@@
 			)
 		)
-		(property "Value" "2k7"
+		(property "Value" "DNP"
 			(at 163.83 111.7599 0)
 			(effects

Commit message: Pokeymax v4_53 as produced
git-svn-id: svn+ssh://192.168.0.3/home/svnfpga/repo/trunk@1512 d6161ac3-aae1-4d52-9b05-ea9ac36b53d3
Parts:
- renumbered R22 to R28, R23 to R29
Changed lines of the file:
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@@
 		(dnp no)
 		(fields_autoplaced yes)
-		(property "Reference" "R22"
+		(property "Reference" "R28"
 			(at 48.26 111.7599 0)
 			(effects
@@
 			(project ""
 				(path "/f8f92944-710a-49a0-a698-f840e5f20e15/473fb442-f6a6-4f3e-b077-9a313beb11d5"
-					(reference "R22")
+					(reference "R28")
 					(unit 1)
 				)
@@
 		(dnp no)
 		(fields_autoplaced yes)
-		(property "Reference" "R23"
+		(property "Reference" "R29"
 			(at 163.83 109.2199 0)
 			(effects
@@
 			(project "pokeymax4_5"
 				(path "/f8f92944-710a-49a0-a698-f840e5f20e15/473fb442-f6a6-4f3e-b077-9a313beb11d5"
-					(reference "R23")
-					(unit 1)
-				)
+					(reference "R29")
+					(unit 1)
+				)
