File: atari_800xl/atari_chips/hardware/pokeymax4_5/level_shifters.kicad_sch (KiCad schematic)
At the start: 2 parts, among them U3 SN74CB3T16211DGVR, U5 SN74CB3T16211DGVR

Commit message: 4.55. Got AI to help me improve a few minor things. Regulator mode, extra decoupling for DAC, distances from edge, gnd/power plane switched, track spacing for a few important lines, bigger cap on 2.5v reg, shorter critical traces on 3.3v reg. Also it double checked the sallen key filter. Switched to the JLCPCB plugin for simpler part management.
Parts:
- U3, U5: LCSC (none) -> C2674751
Changed lines of the file:
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@@
+			)
+		)
+		(property "LCSC" "C2674751"
+			(at 184.15 57.15 0)
+			(hide yes)
+			(show_name no)
+			(do_not_autoplace no)
+			(effects
+				(font
+					(size 1.27 1.27)
+				)
 			)
 		)
@@
 			(at 58.42 57.15 0)
 			(hide yes)
+			(show_name no)
+			(do_not_autoplace no)
+			(effects
+				(font
+					(size 1.27 1.27)
+				)
+			)
+		)
+		(property "LCSC" "C2674751"
+			(at 58.42 57.15 0)
+			(hide yes)
