File: atari_800xl/atari_chips/hardware/pokeymax4_5/power.kicad_sch (KiCad schematic)
At the start: 18 parts

Commit message: kicad 10 upgrade
Parts:
- U1, U6: value ~ -> (none)

Commit message: 4.55. Got AI to help me improve a few minor things. Regulator mode, extra decoupling for DAC, distances from edge, gnd/power plane switched, track spacing for a few important lines, bigger cap on 2.5v reg, shorter critical traces on 3.3v reg. Also it double checked the sallen key filter. Switched to the JLCPCB plugin for simpler part management.
Parts:
- added C30: 0.1uF, Capacitor_SMD:C_0402_1005Metric, symbol Device:C
- C10: LCSC (none) -> C1525
- C11: LCSC (none) -> C86295
- C15, C16, C18, C19, C22, C23, C24, C3: LCSC (none) -> C14663
- C2: value 0.1uF -> 2u2; LCSC (none) -> C23630
- C26: LCSC (none) -> C23630
- C27: LCSC (none) -> C19666
- FB1: LCSC (none) -> C19330
- L1: LCSC (none) -> C171753
- R17: value 10 -> 33; LCSC (none) -> C23140
- U1: LCSC (none) -> C622555
- U6: LCSC (none) -> C398923
Connections:
- net +3.3V: now also C30.1
- net +5V: now also U6.1 (MODE)
- net GND: now also C30.2; no longer U6.1 (MODE)
